Commit message: edited urdf to include a fixed link.
edited urdf to include a fixed link. this fixed link allows the end effector point used by trajectory tracking to be at the desired location rather than the previous wrist_3_joint origin. Other files were also edited to reflect this change.

File: urdf/Arm_V2_edited_2.urdf (robot description, URDF)
Before this commit: robot Arm_V2_edited_2, 11 links, 10 joints
Links:
- removed link wrist_1_link
- removed link wrist_2_link
- removed link wrist_3_link
- added link tip_link, mass 0.0195; collision mesh filename=package://arm_v2_description/meshes/tip_link.STL; visual mesh filename=package://arm_v2_description/meshes/tip_link.STL
- added link wrist_link_1, mass 0.132446543816184; collision mesh filename=package://arm_v2_description/meshes/wrist_link_1.STL; visual mesh filename=package://arm_v2_description/meshes/wrist_link_1.STL
- added link wrist_link_2, mass 0.110570086754039; collision mesh filename=package://arm_v2_description/meshes/wrist_link_2.STL; visual mesh filename=package://arm_v2_description/meshes/wrist_link_2.STL
- added link wrist_link_3, mass 0.175480660661564; collision mesh filename=package://arm_v2_description/meshes/wrist_link_3.STL; visual mesh filename=package://arm_v2_description/meshes/wrist_link_3.STL
Joints:
- removed joint wrist_1_joint
- removed joint wrist_2_joint
- removed joint wrist_3_joint
- added joint tip_fixed_joint: type fixed, parent wrist_link_3, child tip_link, origin xyz=0.06 -0.0325 0 rpy=0 0 0, axis 0 0 0
- added joint wrist_joint_1: type revolute, parent high_link_4, child wrist_link_1, origin xyz=0.05 0 0.02 rpy=0 0 0, axis 0 1 0, limit lower=-3.1416 upper=3.1416 effort=0 velocity=0
- added joint wrist_joint_2: type continuous, parent wrist_link_1, child wrist_link_2, origin xyz=0.043 -0.0325 0 rpy=0 0 0, axis 1 0 0, limit lower=-3.1416 upper=3.1416 effort=0 velocity=0
- added joint wrist_joint_3: type revolute, parent wrist_link_2, child wrist_link_3, origin xyz=0.0631 0.0325 0 rpy=0 0 0, axis 0 1 0, limit lower=-3.1416 upper=3.1416 effort=0 velocity=0
