Commit message: version for reading all 6 joints
finalized version for reading all 6 joints

File: urdf/Arm_V2_edited_2.urdf (robot description, URDF)
Before this commit: robot Arm_V2_urdf_with_fixed_joint, 12 links, 11 joints
Links:
- link high_link_2: mass 0.110507990252835 -> 0.110507990252836
- link high_link_3: mass 0.110507990252836 -> 0.110507990252835
- link low_link_2: mass 0.110507990252835 -> 0.110507990252836
- link low_link_3: mass 0.110507990252836 -> 0.110507990252835
- link wrist_link_3: mass 0.175480660661564 -> 0.297698869950329
Joints:
- joint tip_fixed_joint: origin xyz=0.06 -0.0325 0 rpy=0 0 0 -> xyz=0.0600000000000021 -0.0324999999999982 0 rpy=0 0 0
- joint wrist_joint_3: origin xyz=0.0631 0.0325 0 rpy=0 0 0 -> xyz=0.0631 0.029478 0.013686 rpy=0 0 0
